Commit message: Added new branch with ROS2 Jazzy and Gazebo Harmonic support

File: install/my_simulation/share/my_simulation/urdf/imu.xacro (robot description, xacro)
@@ -1,34 +1 @@
-<?xml version="1.0"?>
-<robot xmlns:xacro="http://www.ros.org/wiki/xacro"  name="robot">
-  <joint name="imu_joint" type="fixed">
-    <origin rpy="0 3.141592653589793 0" xyz="0 0 0"/>
-    <parent link="base_link"/>
-    <child link="imu_link"/>
-  </joint>
-  <link name="imu_link">
-    <inertial>
-      <origin xyz="0 0 0"/>
-      <mass value="0.005"/>
-      <inertia ixx="1.67e-8" ixy="0" ixz="0" iyy="1.67e-8" iyz="0" izz="1.67e-8"/>
-    </inertial>
-  </link>
-  <gazebo reference="imu_link">
-    <gravity>true</gravity>
-    <sensor name="imu_sensor" type="imu">
-      <always_on>true</always_on>
-      <update_rate>200</update_rate>
-      <visualize>true</visualize>
-      <pose>0 0 0 0 0 0</pose>
-      <plugin filename="libgazebo_ros_imu_sensor.so" name="imu_plugin">
-        <topicName>imu_raw</topicName>
-        <update_rate>0</update_rate>
-        <bodyName>imu_link</bodyName>
-        <gaussianNoise>0.0</gaussianNoise>
-        <xyzOffset>0 0 0</xyzOffset>
-        <rpyOffset>0 0 0</rpyOffset>
-        <frameName>base_link</frameName>
-        <initialOrientationAsReference>false</initialOrientationAsReference>
-      </plugin>
-    </sensor>
-  </gazebo>
-</robot>
+/home/gro5293/ros2-lidar/src/my_simulation/urdf/imu.xacro

File: install/my_simulation/share/my_simulation/urdf/lidar.xacro (robot description, xacro)
@@ -1,77 +1 @@
-<?xml version="1.0"?>
-<robot xmlns:xacro="http://www.ros.org/wiki/xacro"  name="robot">
-    <!-- Change it to choose the lidar parameters from Ouster OS1 or other -->
-    <xacro:property name="lidar_model" value="ouster"/>
-    <xacro:arg name="lidar_base_offset_z" default="0.205"/>
-    <xacro:arg name="lidar_inclination" default="${pi/4}"/>
-    <xacro:macro name="cylinder_inertia" params="m r h">
-        <inertial>
-        <origin xyz="0 0 0" rpy="${pi/2} 0 0" />
-        <mass value="${m}"/>
-        <inertia ixx="${(m/12) * (3*r*r + h*h)}" ixy = "0" ixz = "0" iyy="${(m/12) * (3*r*r + h*h)}" iyz = "0" izz="${(m/2) * (r*r)}"/>
-        </inertial>
-    </xacro:macro>
-    <xacro:macro name="lidar_parameters" params="samp res min_ang max_ang">
-        <samples>${samp}</samples>
-        <resolution>${res}</resolution>
-        <min_angle>${min_ang}</min_angle>
-        <max_angle>${max_ang}</max_angle>
-    </xacro:macro>
-    <joint name="lidar_base_joint" type="fixed">
-        <parent link="base_link"/>
-        <child link="lidar_link"/>
-        <origin xyz="0 0 $(arg lidar_base_offset_z)" rpy="0 $(arg lidar_inclination) 0"/>
-    </joint>
-    <link name="lidar_link">
-        <visual>
-            <origin xyz="0 0 0" rpy="0 0 0"/>
-            <geometry>
-                <cylinder length="0.05" radius="0.05"/>
-            </geometry>
-            <material name="red">
-                <color rgba="1 0 0 1.0"/>
-            </material>
-        </visual>
-        <collision>
-            <geometry>
-                <cylinder length="0.05" radius="0.05"/>
-            </geometry>
-        </collision>
-        <xacro:cylinder_inertia m="0.1" r="0.05" h="0.05"/>
-    </link>
-    <gazebo reference="lidar_link">
-        <material>Gazebo/Red</material>
-        <sensor name="ouster-OS0" type="ray">
-            <pose>0 0 0 0 0 0</pose>
-            <visualize>false</visualize>
-            <update_rate>0.25</update_rate>
-            <ray>
-                <scan>
-                    <horizontal>
-                        <xacro:if value="${lidar_model == 'ouster'}">
-                            <!-- Set 'samp'=1024 for a real Ouster Lidar parameter, it was set to 64 to make the simulation run faster -->
-                            <xacro:lidar_parameters samp="250" res="1" min_ang="${-pi*2}" max_ang="${pi*2}"/>
-                        </xacro:if>
-                    </horizontal>
-                    <vertical>
-                        <xacro:if value="${lidar_model == 'ouster'}">
-                            <xacro:lidar_parameters samp="32" res="1" min_ang="${-pi/4}" max_ang="${pi/4}"/>
-                        </xacro:if>
-                    </vertical>
-                </scan>
-                <range>
-                    <min>0.25</min> <!-- Min distance in meters -->
-                    <max>1.5</max> <!-- Max distance in meters -->
-                    <resolution>0.001</resolution>
-                </range>
-            </ray>
-            <plugin name="lidar" filename="libgazebo_ros_ray_sensor.so">
-                <output_type>sensor_msgs/PointCloud2</output_type>
-                <frame_name>lidar_link</frame_name>
-                <organize_cloud>false</organize_cloud>
-                <min_range>0.9</min_range>
-                <max_range>50.0</max_range>
-            </plugin>
-        </sensor>
-    </gazebo>
-</robot>
+/home/gro5293/ros2-lidar/src/my_simulation/urdf/lidar.xacro

File: install/my_simulation/share/my_simulation/urdf/only_lidar/base_core.xacro (robot description, xacro)
@@ -1,16 +1 @@
-<?xml version="1.0"?>
-<robot name="robot_core" xmlns:xacro="http://ros.org/wiki/xacro">
-  <!-- Robot Base link -->
-  <!-- The base link is empty because it can't have inertia parameters
-   to run correctly in Gazebo and also because is a ROS standard to
-   always have a 'base_link' -->
-  <link name="world">
-  </link>
-  <link name="base_link">
-  </link>
-  <joint name="base_to_world_joint" type="fixed">
-    <parent link="world"/>
-    <child link="base_link"/>
-    <origin xyz="0 0 0" rpy="0 0 0"/>
-  </joint>
-</robot>
+/home/gro5293/ros2-lidar/src/my_simulation/urdf/only_lidar/base_core.xacro

File: install/my_simulation/share/my_simulation/urdf/only_lidar/only_lidar.urdf.xacro (robot description, xacro)
@@ -1,7 +1 @@
-<?xml version="1.0"?>
-<robot xmlns:xacro="http://www.ros.org/wiki/xacro"  name="robot">
-    <xacro:arg name="lidar_base_offset_z" default="1"/>
-    <xacro:include filename="base_core.xacro" />
-    <xacro:include filename="../lidar.xacro"/>
-    <xacro:include filename="../imu.xacro" />
-</robot>
+/home/gro5293/ros2-lidar/src/my_simulation/urdf/only_lidar/only_lidar.urdf.xacro

File: install/my_simulation/share/my_simulation/urdf/robot.urdf.xacro (robot description, xacro)
@@ -1,6 +1 @@
-<?xml version="1.0"?>
-<robot xmlns:xacro="http://www.ros.org/wiki/xacro"  name="robot">
-    <xacro:include filename="robot_core.xacro" />
-    <xacro:include filename="lidar.xacro"/>
-    <xacro:include filename="imu.xacro" />
-</robot>
+/home/gro5293/ros2-lidar/src/my_simulation/urdf/robot.urdf.xacro

File: install/my_simulation/share/my_simulation/urdf/robot_core.xacro (robot description, xacro)
@@ -1,148 +1 @@
-<?xml version="1.0"?>
-<robot name="robot_core" xmlns:xacro="http://ros.org/wiki/xacro">
-<xacro:property name="base_width" value = "0.31"/>
-<xacro:property name="base_length" value = "0.42"/>
-<xacro:property name="base_height" value = "0.18"/>
-<xacro:property name="wheel_radius" value="0.10"/>
-<xacro:property name="wheel_width" value="0.04"/>
-<xacro:property name="wheel_ygap" value="0.025"/>
-<xacro:property name="wheel_zoff" value="0.01"/>
-<xacro:property name="wheel_xoff" value="0.05"/>
-<xacro:property name="caster_xoff" value="0.1"/>
-  <!-- Define intertial property macros  -->
-  <xacro:macro name="box_inertia" params="m w h d">
-    <inertial>
-      <origin xyz="0 0 0" rpy="${pi/2} 0 ${pi/2}"/>
-      <mass value="${m}"/>
-      <inertia ixx="${(m/12) * (h*h + d*d)}" ixy="0.0" ixz="0.0" iyy="${(m/12) * (w*w + d*d)}" iyz="0.0" izz="${(m/12) * (w*w + h*h)}"/>
-    </inertial>
-  </xacro:macro>
-  <xacro:macro name="cylinder_inertia" params="m r h">
-    <inertial>
-      <origin xyz="0 0 0" rpy="${pi/2} 0 0" />
-      <mass value="${m}"/>
-      <inertia ixx="${(m/12) * (3*r*r + h*h)}" ixy = "0" ixz = "0" iyy="${(m/12) * (3*r*r + h*h)}" iyz = "0" izz="${(m/2) * (r*r)}"/>
-    </inertial>
-  </xacro:macro>
-  <xacro:macro name="sphere_inertia" params="m r">
-    <inertial>
-      <mass value="${m}"/>
-      <inertia ixx="${(2/5) * m * (r*r)}" ixy="0.0" ixz="0.0" iyy="${(2/5) * m * (r*r)}" iyz="0.0" izz="${(2/5) * m * (r*r)}"/>
-    </inertial>
-  </xacro:macro>
-  <!-- Base footprint necessary for rtabmap to work
-  <link name="base_footprint"/>
-  <joint name="base_footprint_joint" type="fixed">
-    <parent link="base_footprint"/>
-    <child link="base_link"/>
-    <origin xyz="0 0 0" rpy="0 0 0"/>
-  </joint>-->
-  <!-- Robot Base link -->
-  <!-- The base link is empty because it can't have inertia parameters
-   to run correctly in Gazebo and also because is a ROS standard to
-   always have a 'base_link' -->
-  <link name="base_link">
-  </link>
-  <!-- Robot Chassis -->
-  <link name="chassis">
-    <visual>
-    <origin xyz="0 0 ${base_height/2}" rpy="0 0 0"/>
-      <geometry>
-        <box size="${base_length} ${base_width} ${base_height}"/>
-      </geometry>
-      <material name="Cyan">
-        <color rgba="0 1.0 1.0 1.0"/>
-      </material>
-    </visual>
-    <collision>
-    <origin xyz="0 0 ${base_height/2}" rpy="0 0 0"/>
-      <geometry>
-        <box size="${base_length} ${base_width} ${base_height}"/>
-      </geometry>
-    </collision>
-    <xacro:box_inertia m="5" w="${base_width}" d="${base_length}" h="${base_height}"/>
-  </link>
-   <gazebo reference="chassis">
-    <material>Gazebo/Orange</material>
-  </gazebo>
-  <joint name="chassis_joint" type="fixed">
-    <parent link="base_link"/>
-    <child link="chassis"/>
-    <origin xyz="0 0 0" rpy="0 0 0"/>
-  </joint>
-    <!-- Caster Wheel -->
-  <link name="caster">
-    <visual>
-      <geometry>
-        <sphere radius="${wheel_zoff}"/>
-      </geometry>
-      <material name="white">
-        <color rgba="1 1.0 1.0 1.0"/>
-      </material>
-    </visual>
-    <collision>
-      <origin xyz="0 0 0" rpy="0 0 0"/>
-      <geometry>
-        <sphere radius="${wheel_zoff}"/>
-      </geometry>
-    </collision>
-    <xacro:sphere_inertia m="0.5" r="${(wheel_radius+wheel_zoff-(base_height/2))}"/>
-  </link>
-   <gazebo reference="caster">
-    <material>Gazebo/Blue</material>
-  </gazebo>
-  <joint name="caster_joint" type="fixed">
-    <parent link="base_link"/>
-    <child link="caster"/>
-    <origin xyz="${-caster_xoff} 0.0 0" rpy="0 0 0"/>
-  </joint>
-    <!-- Wheels -->
-  <xacro:macro name="wheel" params="prefix x_reflect y_reflect">
-    <link name="${prefix}_link">
-      <visual>
-        <origin xyz="0 0 0" rpy="${pi/2} 0 0"/>
-        <geometry>
-            <cylinder radius="${wheel_radius}" length="${wheel_width}"/>
-        </geometry>
-        <material name="Gray">
-          <color rgba="0.5 0.5 0.5 1.0"/>
-        </material>
-      </visual>
-      <collision>
-        <origin xyz="0 0 0" rpy="${pi/2} 0 0"/>
-        <geometry>
-          <cylinder radius="${wheel_radius}" length="${wheel_width}"/>
-        </geometry>
-      </collision>
-      <xacro:cylinder_inertia m="0.5" r="${wheel_radius}" h="${wheel_width}"/>
-    </link>
-    <joint name="${prefix}_joint" type="continuous">
-      <parent link="base_link"/>
-      <child link="${prefix}_link"/>
-      <origin xyz="${-x_reflect*wheel_xoff} ${y_reflect*(base_width/2+wheel_ygap)} ${wheel_radius-wheel_zoff}" rpy="0 0 0"/>
-      <axis xyz="0 1 0"/>
-    </joint>
-  </xacro:macro>
-  <xacro:wheel prefix="drivewhl_l" x_reflect="-1" y_reflect="1" />
-  <xacro:wheel prefix="drivewhl_r" x_reflect="-1" y_reflect="-1" />
-  <!-- Gazebo plugins that provide robot control -->
-  <gazebo>
-  <plugin name='diff_drive' filename='libgazebo_ros_diff_drive.so'>
-    <!-- wheels -->
-    <left_joint>drivewhl_l_joint</left_joint>
-    <right_joint>drivewhl_r_joint</right_joint>
-    <!-- kinematics -->
-    <wheel_separation>${2*(base_width/2+wheel_ygap)}</wheel_separation>
-    <wheel_diameter>${wheel_radius*2}</wheel_diameter>
-    <!-- limits -->
-    <max_wheel_torque>80</max_wheel_torque>
-    <max_wheel_acceleration>1.0</max_wheel_acceleration>
-    <!-- output -->
-    <publish_odom>true</publish_odom>
-    <publish_odom_tf>true</publish_odom_tf>
-    <publish_wheel_tf>true</publish_wheel_tf>
-    <odometry_frame>odom</odometry_frame>
-    <robot_base_frame>base_link</robot_base_frame>
-  </plugin>
-</gazebo>
-</robot>
+/home/gro5293/ros2-lidar/src/my_simulation/urdf/robot_core.xacro

File: src/my_simulation/urdf/imu.xacro (robot description, xacro)
@@ -1,4 +1,4 @@
 <?xml version="1.0"?>
-<robot xmlns:xacro="http://www.ros.org/wiki/xacro"  name="robot">
+<robot xmlns:xacro="http://www.ros.org/wiki/xacro" name="robot">
   <joint name="imu_joint" type="fixed">
     <origin rpy="0 3.141592653589793 0" xyz="0 0 0"/>
@@ -14,21 +14,24 @@
   </link>
   <gazebo reference="imu_link">
-    <gravity>true</gravity>
-    <sensor name="imu_sensor" type="imu">
+    <plugin name="gz::sim::systems::Imu" filename="gz-sim-imu-system">
+      <ros>
+        <remapping>imu:=/imu</remapping>
+      </ros>
+      <frame_id>base_link</frame_id>
+      <update_rate>200</update_rate>
       <always_on>true</always_on>
-      <update_rate>200</update_rate>
       <visualize>true</visualize>
-      <pose>0 0 0 0 0 0</pose>
-      <plugin filename="libgazebo_ros_imu_sensor.so" name="imu_plugin">
-        <topicName>imu_raw</topicName>
-        <update_rate>0</update_rate>
-        <bodyName>imu_link</bodyName>
-        <gaussianNoise>0.0</gaussianNoise>
-        <xyzOffset>0 0 0</xyzOffset>
-        <rpyOffset>0 0 0</rpyOffset>
-        <frameName>base_link</frameName>
-        <initialOrientationAsReference>false</initialOrientationAsReference>
-      </plugin>
-    </sensor>
+      <orientation_reference_frame>world</orientation_reference_frame>
+      <noise>
+        <angular_velocity>
+          <mean>0.0</mean>
+          <stddev>0.0</stddev>
+        </angular_velocity>
+        <linear_acceleration>
+          <mean>0.0</mean>
+          <stddev>0.0</stddev>
+        </linear_acceleration>
+      </noise>
+    </plugin>
   </gazebo>
 </robot>

File: src/my_simulation/urdf/lidar.xacro (robot description, xacro)
@@ -1,77 +1,85 @@
 <?xml version="1.0"?>
-<robot xmlns:xacro="http://www.ros.org/wiki/xacro"  name="robot">
-    <!-- Change it to choose the lidar parameters from Ouster OS1 or other -->
-    <xacro:property name="lidar_model" value="ouster"/>
-    <xacro:arg name="lidar_base_offset_z" default="0.205"/>
-    <xacro:arg name="lidar_inclination" default="${pi/4}"/>
-    <xacro:macro name="cylinder_inertia" params="m r h">
-        <inertial>
-        <origin xyz="0 0 0" rpy="${pi/2} 0 0" />
-        <mass value="${m}"/>
-        <inertia ixx="${(m/12) * (3*r*r + h*h)}" ixy = "0" ixz = "0" iyy="${(m/12) * (3*r*r + h*h)}" iyz = "0" izz="${(m/2) * (r*r)}"/>
-        </inertial>
-    </xacro:macro>
-    <xacro:macro name="lidar_parameters" params="samp res min_ang max_ang">
-        <samples>${samp}</samples>
-        <resolution>${res}</resolution>
-        <min_angle>${min_ang}</min_angle>
-        <max_angle>${max_ang}</max_angle>
-    </xacro:macro>
-    <joint name="lidar_base_joint" type="fixed">
-        <parent link="base_link"/>
-        <child link="lidar_link"/>
-        <origin xyz="0 0 $(arg lidar_base_offset_z)" rpy="0 $(arg lidar_inclination) 0"/>
-    </joint>
-    <link name="lidar_link">
-        <visual>
-            <origin xyz="0 0 0" rpy="0 0 0"/>
-            <geometry>
-                <cylinder length="0.05" radius="0.05"/>
-            </geometry>
-            <material name="red">
-                <color rgba="1 0 0 1.0"/>
-            </material>
-        </visual>
-        <collision>
-            <geometry>
-                <cylinder length="0.05" radius="0.05"/>
-            </geometry>
-        </collision>
-        <xacro:cylinder_inertia m="0.1" r="0.05" h="0.05"/>
-    </link>
-    <gazebo reference="lidar_link">
-        <material>Gazebo/Red</material>
-        <sensor name="ouster-OS0" type="ray">
-            <pose>0 0 0 0 0 0</pose>
-            <visualize>false</visualize>
-            <update_rate>0.25</update_rate>
-            <ray>
-                <scan>
-                    <horizontal>
-                        <xacro:if value="${lidar_model == 'ouster'}">
-                            <!-- Set 'samp'=1024 for a real Ouster Lidar parameter, it was set to 64 to make the simulation run faster -->
-                            <xacro:lidar_parameters samp="250" res="1" min_ang="${-pi*2}" max_ang="${pi*2}"/>
-                        </xacro:if>
-                    </horizontal>
-                    <vertical>
-                        <xacro:if value="${lidar_model == 'ouster'}">
-                            <xacro:lidar_parameters samp="32" res="1" min_ang="${-pi/4}" max_ang="${pi/4}"/>
-                        </xacro:if>
-                    </vertical>
-                </scan>
-                <range>
-                    <min>0.25</min> <!-- Min distance in meters -->
-                    <max>1.5</max> <!-- Max distance in meters -->
-                    <resolution>0.001</resolution>
-                </range>
-            </ray>
-            <plugin name="lidar" filename="libgazebo_ros_ray_sensor.so">
-                <output_type>sensor_msgs/PointCloud2</output_type>
-                <frame_name>lidar_link</frame_name>
-                <organize_cloud>false</organize_cloud>
-                <min_range>0.9</min_range>
-                <max_range>50.0</max_range>
-            </plugin>
-        </sensor>
-    </gazebo>
+<robot xmlns:xacro="http://www.ros.org/wiki/xacro" name="robot">
+  <xacro:property name="lidar_model" value="ouster-os0"/>
+  <xacro:arg name="lidar_base_offset_z" default="0.205"/>
+  <xacro:arg name="lidar_inclination" default="${pi/4}"/>
+  <xacro:macro name="cylinder_inertia" params="m r h">
+    <inertial>
+      <origin xyz="0 0 0" rpy="${pi/2} 0 0"/>
+      <mass value="${m}"/>
+      <inertia
+        ixx="${(m/12)*(3*r*r + h*h)}"
+        ixy="0" ixz="0"
+        iyy="${(m/12)*(3*r*r + h*h)}"
+        iyz="0"
+        izz="${(m/2)*(r*r)}"/>
+    </inertial>
+  </xacro:macro>
+  <xacro:macro name="lidar_parameters" params="samp res min_ang max_ang">
+    <samples>${samp}</samples>
+    <resolution>${res}</resolution>
+    <min_angle>${min_ang}</min_angle>
+    <max_angle>${max_ang}</max_angle>
+  </xacro:macro>
+  <joint name="lidar_base_joint" type="fixed">
+    <parent link="base_link"/>
+    <child link="lidar_link"/>
+    <origin xyz="0 0 $(arg lidar_base_offset_z)" rpy="0 $(arg lidar_inclination) 0"/>
+  </joint>
+  <link name="lidar_link">
+    <visual>
+      <origin xyz="0 0 0" rpy="0 0 0"/>
+      <geometry>
+        <cylinder length="0.05" radius="0.05"/>
+      </geometry>
+      <material name="red">
+        <color rgba="1 0 0 1.0"/>
+      </material>
+    </visual>
+    <collision>
+      <geometry>
+        <cylinder length="0.05" radius="0.05"/>
+      </geometry>
+    </collision>
+    <xacro:cylinder_inertia m="0.1" r="0.05" h="0.05"/>
+  </link>
+  <gazebo>
+    <plugin filename="gz-sim-sensors-system" name="gz::sim::systems::Sensors">
+      <render_engine>ogre2</render_engine>
+    </plugin>
+  </gazebo>
+  <gazebo reference="lidar_link">
+    <sensor name="gpu_lidar" type="gpu_lidar">
+      <topic>/lidar</topic>
+      <gz_frame_id>lidar_link</gz_frame_id>
+      <update_rate>0.25</update_rate>
+      <lidar>
+        <scan>
+          <horizontal>
+            <xacro:if value="${lidar_model == 'ouster-os0'}">
+              <!-- Set 'samp'=1024 for a real Ouster Lidar parameter, it was set to 64 to make the simulation run faster -->
+              <xacro:lidar_parameters samp="250" res="1" min_ang="${-pi*2}" max_ang="${pi*2}"/>
+            </xacro:if>
+          </horizontal>
+          <vertical>
+            <xacro:if value="${lidar_model == 'ouster-os0'}">
+              <xacro:lidar_parameters samp="32" res="1" min_ang="${-pi/4}" max_ang="${pi/4}"/>
+            </xacro:if>
+          </vertical>
+        </scan>
+        <range>
+          <min>0.25</min> <!-- Min distance in meters -->
+          <max>100</max> <!-- Max distance in meters -->
+          <resolution>0.01</resolution>
+        </range>
+        <!--<noise>
+          <type>gaussian</type>
+          <mean>0.0</mean>
+          <stddev>0.01</stddev>
+        </noise>-->
+      </lidar>
+      <always_on>true</always_on>
+      <visualize>false</visualize>
+    </sensor>
+  </gazebo>
 </robot>

File: src/my_simulation/urdf/robot_core.xacro (robot description, xacro)
@@ -128,21 +128,32 @@
   <!-- Gazebo plugins that provide robot control -->
   <gazebo>
-  <plugin name='diff_drive' filename='libgazebo_ros_diff_drive.so'>
-    <!-- wheels -->
-    <left_joint>drivewhl_l_joint</left_joint>
-    <right_joint>drivewhl_r_joint</right_joint>
-    <!-- kinematics -->
-    <wheel_separation>${2*(base_width/2+wheel_ygap)}</wheel_separation>
-    <wheel_diameter>${wheel_radius*2}</wheel_diameter>
-    <!-- limits -->
-    <max_wheel_torque>80</max_wheel_torque>
-    <max_wheel_acceleration>1.0</max_wheel_acceleration>
-    <!-- output -->
-    <publish_odom>true</publish_odom>
-    <publish_odom_tf>true</publish_odom_tf>
-    <publish_wheel_tf>true</publish_wheel_tf>
-    <odometry_frame>odom</odometry_frame>
-    <robot_base_frame>base_link</robot_base_frame>
-  </plugin>
-</gazebo>
+    <plugin filename="gz-sim-diff-drive-system" name="gz::sim::systems::DiffDrive">
+      <!-- joints -->
+      <left_joint>drivewhl_l_joint</left_joint>
+      <right_joint>drivewhl_r_joint</right_joint>
+      <!-- geometry -->
+      <wheel_separation>${2*(base_width/2+wheel_ygap)}</wheel_separation>
+      <wheel_radius>${wheel_radius}</wheel_radius>
+      <!-- frames -->
+      <odom_frame>odom</odom_frame>
+      <robot_base_frame>base_link</robot_base_frame>
+      <topic>/cmd_vel</topic>
+      <!-- limits -->
+      <max_linear_acceleration>1.0</max_linear_acceleration>
+      <max_angular_acceleration>1.0</max_angular_acceleration>
+    </plugin>
+    <plugin filename="gz-sim-odometry-publisher-system" name="gz::sim::systems::OdometryPublisher">
+        <odom_frame>odom</odom_frame>
+        <robot_base_frame>base_link</robot_base_frame>
+        <odom_publish_frequency>50</odom_publish_frequency>
+        <odom_topic>/odom</odom_topic>
+        <tf_topic>/tf</tf_topic>
+        <dimensions>2</dimensions>
+    </plugin>
+    <plugin filename="gz-sim-joint-state-publisher-system" name="gz::sim::systems::JointStatePublisher">
+      <topic>joint_states</topic>
+      <joint_name>drivewhl_r_joint</joint_name>
+      <joint_name>drivewhl_l_joint</joint_name>
+    </plugin>
+  </gazebo>
 </robot>
